File: BoardSheme.sch (EAGLE design)
At the start: 25 parts, among them IC1 7805DT, Q1 IRF540, Q2 IRF540, Q3 IRF540, Q4 IRF540, Q5 IRF540, Q6 IRF540

Commit message: V0.1 completed
Parts:
- added S2, S3, S4, S5, S6, S7: (no value), SparkFun-Switches:SWITCH-SPDT-PTH-11.6X4.0MM
Connections:
- new net N$20: RIGHTPAD.1
- net +5V: now also S2.P, S3.P, S4.P, S5.P, S6.P, S7.P
- net N$10: now also S4.S
- net N$11: now also S5.S
- net N$12: now also S6.S
- net N$13: now also S7.S
- net N$14: now also R3.1, RIGHTPAD.4; no longer R1.1, RIGHTPAD.1
- net N$15: now also RIGHTPAD.3; no longer RIGHTPAD.2
- net N$16: now also R1.1, RIGHTPAD.2; no longer R3.1, RIGHTPAD.3
- net N$17: now also RIGHTPAD.5; no longer RIGHTPAD.4
- net N$18: now also RIGHTPAD.8; no longer RIGHTPAD.5
- net N$19: now also RIGHTPAD.9; no longer RIGHTPAD.8
- net N$2: now also S2.S
- net N$9: now also S3.S
